File: AFE_V3/AFE_V3.kicad_pcb (KiCad board)
At the start: 2 copper layers, 220 x 125 mm, 310 parts, among them IC1 AD5141BCPZ100-RL7, IC10 MAX4526EUA+, IC11 TPS7A3001DGNR, IC12 TPS7A4901DGNR, IC13 TPS72325DBVR, IC14 ADP150AUJZ-2.5-R7, IC15 ADP150AUJZ-3.3-R7, IC16 USB3300-EZK-TR, IC17 STMPS2151MTR, IC2 OPA189ID, IC3 OPA189ID, IC4 OPA189ID, IC5 OPA189ID, IC6 LT6372HMSE-1#PBF, IC7 MAX4526EUA+, IC8 MAX4526EUA+, IC9 MAX4526EUA+, J1 Conn_Coaxial, J10 Conn_Coaxial, J11 Conn_Coaxial, J12 Conn_Coaxial, J13 DEBUG_01x04, J14 TO_SWITCH, J2 USB_C_Receptacle_USB2.0_16P, J3 DS-201, J4 DEBUG_01x04, J5 Conn_01x07, J6 Conn_Coaxial, J7 Conn_Coaxial, J8 Conn_Coaxial, J9 Conn_Coaxial, Q1 BT137S-600, SW1 KLS7-TS6606-13.0, SW2 KLS7-TS6606-13.0, U1 STM32F407ZETx, U10 STM32F103C8Tx, U11 TPC5160-VS2R, U12 TPC5160-VS2R, U2 MDD01N-12, U3 A1215S-1WR3, U4 B1212LS-1WR3, U5 L7905, U6 L7805, U7 AMS1117-3.3, U8 USBLC6-2SC6, U9 HG24LC64M, Y1 Crystal_GND24, Y2 NX3225GD-8MHz, Y3 NX3225GD-8MHz, Y4 X321532768KJD2SI-32.768

Commit message: Started pcb placing
Parts:
- C100, C101, C108, C109, C110, C111, C114, C115, C116, C118, C120, C121, C94, C95, C96, C97, C98, C99, IC11, IC12: moved to B.Cu
- moved U7 192.2 mm to (70.0, 224.2), turned to 90 degrees
- moved C116 189.9 mm to (145.0, 263.0), turned to -90 degrees
- moved U4 188.2 mm to (79.2, 236.4), turned to 90 degrees
- moved U3 186.3 mm to (118.5, 236.9), turned to -90 degrees
- moved C117 186.1 mm to (153.7, 262.4), turned to -90 degrees
- moved C108 181.3 mm to (122.5, 252.5), turned to 180 degrees
- moved C118 178.4 mm to (145.0, 257.5), turned to -90 degrees
- moved C105 177.7 mm to (122.6, 263.0), turned to 180 degrees
- moved C119 175.1 mm to (153.5, 257.5), turned to -90 degrees
- moved C115 173.4 mm to (134.0, 264.0), turned to 180 degrees
- moved C114 171.4 mm to (136.6, 259.2)
- moved C99 170.8 mm to (121.5, 248.5), turned to -90 degrees
- moved U6 169.0 mm to (139.5, 259.2)
- moved R23 168.6 mm to (119.1, 265.0), turned to 180 degrees
- moved C106 168.3 mm to (126.0, 258.5), turned to 90 degrees
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Routing:
- added copper zone on B.Cu, net GNDPWR
- added copper zone on F.Cu, net GNDPWR

Commit message: PCB tracing in progress. Added some 3d models
Parts:
- removed C138: 100n/6.3V, Capacitor_SMD:C_0402_1005Metric
- removed C53, C56: 10uF/35V, Capacitor_SMD:C_0805_2012Metric_Pad1.18x1.45mm_HandSolder
- removed C54, C55: 1uF/35V, Capacitor_SMD:C_0603_1608Metric_Pad1.08x0.95mm_HandSolder
- removed D3, D4: TPC5160, zpc-lib:VS2MSOP-10-A_TPK
- removed DA11, DA12: RS3112XK-2.5, Package_SO:SOIC-8_3.9x4.9mm_P1.27mm
- removed DA13, DA7: TPA1286U, Package_SO:MSOP-8_3x3mm_P0.65mm
- removed DA14: RS8651X, Package_SO:SOIC-8_3.9x4.9mm_P1.27mm
- removed JP10, JP11, JP12, JP13, JP14, JP3, JP8, JP9: SolderJumper_2_Open, Jumper:SolderJumper-2_P1.3mm_Open_TrianglePad1.0x1.5mm
- removed the R20 at (284.2, 47.2)
- removed R33, R34: 8.2k, Resistor_SMD:R_0603_1608Metric_Pad0.98x0.95mm_HandSolder
- removed U9: HG24LC64M, Package_SO:SOIC-8_3.9x4.9mm_P1.27mm
- added DA3: RS3112XK-2.5, Package_SO:SOIC-8_3.9x4.9mm_P1.27mm, F.Cu at (461.2, 100.1)
- added DA5: RS3112XK-2.5, Package_SO:SOIC-8_3.9x4.9mm_P1.27mm, F.Cu at (492.4, 194.1)
- added R36: 680, Resistor_SMD:R_0603_1608Metric_Pad0.98x0.95mm_HandSolder, F.Cu at (71.3, 189.5)
- added R37: 680, Resistor_SMD:R_0603_1608Metric_Pad0.98x0.95mm_HandSolder, F.Cu at (73.2, 189.5)
- C123, C124, C125, C126, C127, C128, C129, C131, C133, C136, C137, C139, C140, C141, C142, C143, C144, C145, C146, C147, C148, C149, C150, C151, C152, C153, C154, C155, C156, C157, C158, C159, C16, C160, C161, C17, C20, C21, C22, C23, C47, C79, D13, FB2, IC17, J5, JP6, JP7, R10, R11, R31, R32, R9, U12: moved to B.Cu
- R17: value 1.8k 0.1% -> 680; footprint Resistor_SMD:R_0805_2012Metric_Pad1.20x1.40mm_HandSolder -> Resistor_SMD:R_0603_1608Metric_Pad0.98x0.95mm_HandSolder
- R21: value 10k -> 680
- moved R26 390.5 mm to (55.5, 223.5), turned to 180 degrees
- moved C122 378.2 mm to (55.5, 221.5)
- moved R28 377.8 mm to (60.3, 216.7)
- moved R27 377.6 mm to (57.9, 209.9), turned to 90 degrees
- moved R29 373.5 mm to (59.6, 209.5), turned to 90 degrees
- moved FB2 369.7 mm to (57.0, 209.9), turned to -90 degrees
- moved C123 367.6 mm to (61.9, 214.2), turned to 90 degrees
- moved R30 366.0 mm to (71.8, 205.9)
- moved C127 360.0 mm to (72.1, 206.6), turned to 180 degrees
- moved C128 357.9 mm to (72.1, 205.0), turned to 180 degrees
- moved R32 356.6 mm to (78.1, 200.8), turned to 180 degrees
- moved R31 356.1 mm to (74.8, 214.8), turned to 90 degrees
- moved C129 355.0 mm to (80.1, 215.0)
- moved C124 354.2 mm to (73.1, 209.2), turned to 90 degrees
- moved C130 352.9 mm to (75.2, 202.5), turned to -90 degrees
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Connections:
- net /USB HS/DM_CONN renamed /USB HS/D_CONN-
- net /USB HS/DP_CONN renamed /USB HS/D_CONN+
- net Net-(J2-SHIELD) renamed /USB HS/USB_SHIELD
- net Net-(U10-VBAT) renamed /MCU_SMALL_VDD
- D17 pad 2: /LED_ERROR -> Net-(D17-A)
- D18 pad 2: /LED_OK -> Net-(D18-A)
- D19 pad 2: /LED_SMALL_ERROR -> Net-(D19-A)
- D20 pad 2: /LED_SMALL_OK -> Net-(D20-A)
- DA6 pad 6: Net-(DA6-OUT) -> /Measurement_all_vars/ADC_REF
- IC16 pad 8: /USB HS/DM -> /USB HS/DN
- IC4 pad 4: GNDA -> -15AVDD
- R17 pad 1: /Measurement_all_vars/Mid_gnd_comp -> Net-(D18-A)
- R17 pad 2: Net-(DA1-RG2) -> /LED_OK
- R21 pad 1: /Measurement_all_vars/SDO_CAL_SPI -> Net-(D17-A)
- R21 pad 2: 3V3AVDD -> /LED_ERROR
- RN1 pad 8: Net-(DA6-OUT) -> Net-(DA3-OUT)
- U1 pad 136: /MEM_SCL -> unconnected-(U1-PB6-Pad136)
- U1 pad 137: /MEM_SDA -> unconnected-(U1-PB7-Pad137)
- U8 pad 4: /USB HS/DP -> /USB HS/DN
- U8 pad 6: /USB HS/DM -> /USB HS/DP
Routing:
- net /USB HS/DN: track 0.00 -> 14.0 mm
- net /USB HS/DP: track 0.00 -> 14.0 mm
- net /USB HS/D_CONN-: track 0.00 -> 10.9 mm
- net /USB HS/D_CONN+: track 0.00 -> 9.90 mm, vias 0 -> 2
Other:
- board size 220 x 125 mm -> 220 x 105.2 mm

Commit message: PCB tracing in progress
Parts:
- removed J10, J11, J12, J6, J7, J8, J9: Conn_Coaxial, Connector_Coaxial:BNC_Amphenol_B6252HB-NPP3G-50_Horizontal
- added C53: 0.1uF/6.3V, Capacitor_SMD:C_0603_1608Metric_Pad1.08x0.95mm_HandSolder, B.Cu at (80.9, 205.5)
- added JP1: SolderJumper_2_Open, Jumper:SolderJumper-2_P1.3mm_Open_TrianglePad1.0x1.5mm, F.Cu at (174.8, 239.7)
- added JP2: SolderJumper_2_Open, Jumper:SolderJumper-2_P1.3mm_Open_TrianglePad1.0x1.5mm, B.Cu at (172.2, 244.9)
- added JP3: SolderJumper_2_Open, Jumper:SolderJumper-2_P1.3mm_Open_TrianglePad1.0x1.5mm, B.Cu at (175.0, 244.9)
- C4, C78, U11: moved to B.Cu
- J1: value Conn_Coaxial -> Conn_2Rows-17Pins; footprint Connector_Coaxial:BNC_Amphenol_B6252HB-NPP3G-50_Horizontal -> Connector_PinHeader_2.54mm:PinHeader_2x08_P2.54mm_Horizontal
- moved U11 422.7 mm to (166.9, 242.4), turned to 180 degrees
- moved DA2 415.4 mm to (180.4, 242.4), turned to 180 degrees
- moved RN1 367.7 mm to (173.0, 243.8), turned to -90 degrees
- moved C6 346.0 mm to (179.1, 247.2), turned to 180 degrees
- moved C78 344.6 mm to (163.3, 239.7), turned to 180 degrees
- moved R2 341.9 mm to (185.5, 243.8), turned to 90 degrees
- moved C9 339.5 mm to (179.1, 237.7), turned to 180 degrees
- moved C3 337.2 mm to (162.1, 244.8), turned to -90 degrees
- moved C5 334.0 mm to (158.8, 238.3), turned to -90 degrees
- moved DA3 327.6 mm to (167.1, 244.2)
- moved C4 325.4 mm to (171.4, 240.2), turned to 90 degrees
- moved DA4 325.0 mm to (163.8, 237.7)
- moved R16 320.4 mm to (192.8, 215.6)
- moved C46 320.2 mm to (168.2, 219.3)
- moved C47 320.2 mm to (177.8, 213.8)
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Connections:
- net Net-(D1-A) renamed /Power/PWR_prot
- net Net-(DA2-REF) renamed /Measurement_all_vars/INA_REF_CAL
- net Net-(DA4-OUT) renamed /Measurement_all_vars/ADC_REF_CAL
- C129 pad 1: /USB HS/1.8VDD -> Net-(IC16-VDD1.8_1)
- D9 pad 3: /CUR+_CH_SEL_MCU -> /CUR-_CH_SEL_MCU
- D9 pad 4: /MEAS+_CH_SEL_MCU -> /MEAS-_CH_SEL_MCU
- D9 pad 5: /MEAS-_CH_SEL_MCU -> /MEAS+_CH_SEL_MCU
- D9 pad 6: /CUR-_CH_SEL_MCU -> /CUR+_CH_SEL_MCU
- IC10 pad 1: Net-(IC10-A) -> imp+1
- IC10 pad 2: Net-(IC10-B) -> imp+2
- IC16 pad 15: /USB HS/1.8VDD -> Net-(IC16-VDD1.8_1)
- IC16 pad 26: /USB HS/1.8VDD -> Net-(IC16-VDD1.8_2)
- IC7 pad 6: Net-(IC7-Y) -> cur+2
- IC7 pad 7: Net-(IC7-X) -> cur+1
- IC8 pad 1: Net-(IC8-A) -> cur-1
- IC8 pad 2: Net-(IC8-B) -> cur-2
- IC9 pad 1: Net-(IC9-A) -> imp-1
- IC9 pad 2: Net-(IC9-B) -> imp-2
- J1 pad 1: Net-(IC7-Y) -> cur+1
- U11 pad 4: GNDA -> Net-(JP2-B)
Routing:
- net 3V3: track 0.00 -> 93.1 mm, vias 0 -> 8
- net /MCU_VDD: track 0.00 -> 87.3 mm, vias 0 -> 11
- net -15AVDD: track 0.00 -> 70.9 mm, vias 0 -> 4
- net +15AVDD: track 0.00 -> 69.8 mm, vias 0 -> 4
- net /ULPI_NXT: track 0.00 -> 62.9 mm, vias 0 -> 2
- net 5AVDD: track 0.00 -> 60.8 mm, vias 0 -> 5
- net /ULPI_DIR: track 0.00 -> 50.2 mm, vias 0 -> 2
- net /ULPI_STP: track 0.00 -> 47.5 mm, vias 0 -> 2
- net cur-2: track 0.00 -> 47.5 mm
- net /ULPI_D7: track 0.00 -> 47.1 mm, vias 0 -> 2
- net cur-1: track 0.00 -> 47.0 mm
- net /USB_RESET: track 0.00 -> 42.4 mm, vias 0 -> 2
- net DGND: track 0.00 -> 40.9 mm, vias 0 -> 20
- net 3V3AVDD: track 0.00 -> 40.5 mm, vias 0 -> 3
- net /Measurement_all_vars/MEAS+: track 0.00 -> 36.0 mm, vias 0 -> 2
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- added copper zone on F.Cu, net /Power/PWR_BUT
- added copper zone on F.Cu, net /Power/PWR_In
- added copper zone on B.Cu, net /Power/PWR_prot
- added copper zone on B.Cu, net DGND
- added copper zone on F.Cu, net DGND
- added copper zone on B.Cu, net GNDA
- added copper zone on F.Cu, net GNDA
Other:
- board size 220 x 105.2 mm -> 193 x 105.2 mm
