File: AFE_V3/Cur_source.kicad_sch (KiCad schematic)
At the start: 60 parts, among them IC1 AD5141BCPZ100-RL7, IC2 OPA189ID, IC3 OPA189ID, IC4 OPA189ID, IC5 OPA189ID, IC7 MAX4526EUA+, J1 Conn_Coaxial, J5 Conn_01x07, J6 Conn_Coaxial

Commit message: PCB tracing in progress. Added some 3d models
Connections:
- net -15AVDD: now also IC4.4 (V-)
- net GNDA: no longer IC4.4 (V-)
Changed lines of the file:
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@@
+	)
+	(junction
+		(at 207.01 142.24)
+		(diameter 0)
+		(color 0 0 0 0)
 	)
 	(junction
@@
 	(junction
 		(at 287.02 96.52)
-		(diameter 0)
-		(color 0 0 0 0)
-	)
-	(junction
-		(at 218.44 142.24)
 		(diameter 0)
 		(color 0 0 0 0)
@@
 	(wire
 		(pts
+			(xy 219.71 139.7) (xy 207.01 139.7)
+		)
+		(stroke
+			(width 0)
+			(type default)
+		)
+	)
+	(wire
+		(pts
 			(xy 154.94 137.16) (xy 163.83 137.16)
 		)
@@
 	(wire
 		(pts
+			(xy 207.01 139.7) (xy 207.01 142.24)
+		)
+		(stroke
+			(width 0)
+			(type default)
+		)
+	)
+	(wire
+		(pts
 			(xy 204.47 208.28) (xy 201.93 208.28)
 		)
@@
 		)
 		(stroke
-			(width 0)
-			(type default)
-		)
-	)
-	(wire
-		(pts
-			(xy 219.71 139.7) (xy 218.44 139.7)
-		)
-		(stroke
-			(width 0)
-			(type default)
-		)
-	)
-	(wire
-		(pts
-			(xy 218.44 139.7) (xy 218.44 142.24)
-		)
-		(stroke

Commit message: PCB tracing in progress
Parts:
- removed J1, J6: Conn_Coaxial, Connector_Coaxial:BNC_Amphenol_B6252HB-NPP3G-50_Horizontal, symbol Connector:Conn_Coaxial
Connections:
- net cur+2: now reaches IC7.6 (Y)
- net cur+1: now reaches IC7.7 (X)
