File: AFE_V3/AFE_V3.kicad_sch (KiCad schematic)
At the start: 73 parts, among them J1 Conn_2Rows-17Pins, J13 DEBUG_01x04, J4 DEBUG_01x04, SW1 KLS7-TS6606-13.0, SW2 KLS7-TS6606-13.0, U1 STM32F407ZETx, U10 STM32F103C8Tx, Y2 NX3225GD-8MHz, Y3 NX3225GD-8MHz, Y4 X321532768KJD2SI-32.768

Commit message: PCB Tracing done. Added CI files
Parts:
- added J6, J7, J8, J9: Screw_Terminal_01x01, MountingHole:MountingHole_3.2mm_M3_Pad_Via, symbol Connector:Screw_Terminal_01x01
Connections:
- net GEN_FSYNC_MCU: now also U1.134 (PB4); no longer U1.44 (PC4)
- net UART_Rx_BIG: now also U1.35 (PA1); no longer U1.102 (PA10)
- net UART_Tx_BIG: now also U1.34 (PA0); no longer U1.101 (PA9)
- net USB_RESET: now also U1.36 (PA2); no longer U1.34 (PA0)
- no-connect marks 111 -> 114

Commit message: Added logo
Parts:
- added HU1, HU2: ~, zpc-lib:SFFF logo, symbol zpc-lib:LOGO
Changed lines of the file:
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@@
+	)
+	(symbol
+		(lib_id "zpc-lib:LOGO")
+		(at 351.79 138.43 0)
+		(unit 1)
+		(exclude_from_sim no)
+		(in_bom yes)
+		(on_board yes)
+		(dnp no)
+		(property "Reference" "HU2"
+			(at 353.06 137.668 0)
+			(effects
+				(font
+					(size 1.27 1.27)
+				)
+				(justify left)
+			)
+		)
+		(property "Value" "~"
+			(at 353.06 139.7 0)
+			(effects
+				(font
+					(size 1.27 1.27)
+				)
+				(justify left)
+			)
+		)
+		(property "Footprint" "zpc-lib:SFFF logo"
+			(at 351.79 138.43 0)
+			(effects
+				(font
+					(size 1.27 1.27)
+				)
+				(hide yes)
+			)
+		)
+		(property "Datasheet" ""
+			(at 351.79 138.43 0)
+			(effects
+				(font
+					(size 1.27 1.27)
+				)
+				(hide yes)
+			)
+		)
+		(property "Description" ""
+			(at 351.79 138.43 0)
+			(effects
+				(font
+					(size 1.27 1.27)
+				)
+				(hide yes)
+			)
+		)
+		(instances
+			(project "AFE_V3"
+				(path "/e9ffbb94-33e2-4158-ac4a-a33b17b122cf"
+					(reference "HU2")
+					(unit 1)
+				)
+			)
+		)
 	)
 	(symbol
@@
 					(unit 1)
 				)
+			)
+		)
+	)
+	(symbol
+		(lib_id "zpc-lib:LOGO")
+		(at 377.19 123.19 0)
+		(unit 1)
+		(exclude_from_sim no)
+		(in_bom yes)
+		(on_board yes)
+		(dnp no)
+		(property "Reference" "HU1"
+			(at 378.46 122.428 0)
+			(effects
+				(font
+					(size 1.27 1.27)
+				)
+				(justify left)
+			)
+		)
+		(property "Value" "~"
+			(at 378.46 124.46 0)
+			(effects
+				(font
+					(size 1.27 1.27)
+				)
+				(justify left)
+			)
+		)
+		(property "Footprint" "zpc-lib:SFFF logo"
+			(at 377.19 123.19 0)
+			(effects
+				(font
+					(size 1.27 1.27)
+				)
+				(hide yes)
+			)
+		)
+		(property "Datasheet" ""
+			(at 377.19 123.19 0)
+			(effects
+				(font
+					(size 1.27 1.27)
+				)
+				(hide yes)
+			)
+		)
+		(property "Description" ""
+			(at 377.19 123.19 0)
+			(effects
+				(font
+					(size 1.27 1.27)
+				)
+				(hide yes)
+			)
+		)
+		(instances
+			(project ""
+				(path "/e9ffbb94-33e2-4158-ac4a-a33b17b122cf"
+					(reference "HU1")
+					(unit 1)
+				)
